File: KiCad/CarSpeedPulser.sch (KiCad schematic (older format))
At the start: 15 parts, among them P1 CONN_01X02, Q1 2SK4017, SW1 RESET, SW2 UP, SW3 DOWN, U1 LPC810, U2 AE-AQM0802, U3 TA48M033F

Commit message: Added writer connector.
Parts:
- added P2: CONN_01X05, Pin_Headers:Pin_Header_Straight_1x05, symbol CONN_01X05
Connections:
- wire segments 47 -> 57
Changed lines of the file:
@@
 L VDD #PWR04
 U 1 1 555A13C5
-P 6800 1600
-F 0 "#PWR04" H 6800 1450 50  0001 C CNN
-F 1 "VDD" H 6800 1750 50  0000 C CNN
-F 2 "" H 6800 1600 60  0000 C CNN
-F 3 "" H 6800 1600 60  0000 C CNN
-	1    6800 1600
+P 7150 1550
+F 0 "#PWR04" H 7150 1400 50  0001 C CNN
+F 1 "VDD" H 7150 1700 50  0000 C CNN
+F 2 "" H 7150 1550 60  0000 C CNN
+F 3 "" H 7150 1550 60  0000 C CNN
+	1    7150 1550
 	1    0    0    -1
 $EndComp
@@
 L AE-AQM0802 U2
 U 1 1 555A2C55
-P 7750 1850
-F 0 "U2" H 7750 1750 50  0000 C CNN
-F 1 "AE-AQM0802" H 7750 2200 50  0000 C CNN
-F 2 "pulser:AE-AQM0802" H 7750 1500 50  0001 C CNN
-F 3 "DOCUMENTATION" H 7750 1400 50  0001 C CNN
-	1    7750 1850
-	1    0    0    -1
-$EndComp
-NoConn ~ 7150 1750
+P 7950 1850
+F 0 "U2" H 7950 1750 50  0000 C CNN
+F 1 "AE-AQM0802" H 7950 2200 50  0000 C CNN
+F 2 "pulser:AE-AQM0802" H 7950 1500 50  0001 C CNN
+F 3 "DOCUMENTATION" H 7950 1400 50  0001 C CNN
+	1    7950 1850
+	1    0    0    -1
+$EndComp
+NoConn ~ 7350 1750
 $Comp
 L PWR_FLAG #FLG06
@@
 	3350 2650 3350 2500
 Wire Wire Line
-	3350 3650 3350 3900
+	3350 3900 3350 3650
 Wire Wire Line
 	2950 3250 2950 3500
@@
 	2950 3800 2950 3900
 Wire Wire Line
-	2650 3900 4800 3900
+	4800 3900 2650 3900
 Connection ~ 3350 3900
 Connection ~ 2950 3450
@@
 	6600 1950 6700 1950
 Wire Wire Line
-	6700 1950 6700 2650
-Wire Wire Line
-	6800 1600 6800 2050
-Wire Wire Line
-	6800 2050 6600 2050
-Wire Wire Line
-	6600 1850 7150 1850
-Wire Wire Line
-	7150 1650 6800 1650
-Connection ~ 6800 1650
-Wire Wire Line
-	6600 2150 6900 2150
-Wire Wire Line
-	6900 2150 6900 1950
-Wire Wire Line
-	6900 1950 7150 1950
-Wire Wire Line
-	7150 2050 7150 2250
-Wire Wire Line
-	7150 2250 6700 2250
+	6700 1350 6700 2650
+Wire Wire Line
+	7150 2050 7150 1550
+Wire Wire Line
+	6600 2050 7150 2050
+Wire Wire Line
+	6600 1850 7350 1850
+Wire Wire Line
+	7350 1650 7150 1650
+Connection ~ 7150 1650
+Wire Wire Line
+	6600 2150 7250 2150
+Wire Wire Line
+	7250 2150 7250 1950
+Wire Wire Line
+	7250 1950 7350 1950
+Wire Wire Line
+	7350 2050 7350 2250
+Wire Wire Line
+	7350 2250 6700 2250
 Wire Wire Line
 	900  1450 900  1500
@@
 	2650 3250 2650 3050
 Wire Wire Line
-	2650 3650 2650 3900
+	2650 3900 2650 3650
 Connection ~ 2950 3900
 $Comp
@@
 Text Label 3600 3150 0    60   ~ 0
 PULSE
+$Comp
+L CONN_01X05 P2
+U 1 1 5559F1FE
+P 5000 950
+F 0 "P2" H 5000 1250 50  0000 C CNN
+F 1 "CONN_01X05" V 5100 950 50  0000 C CNN
+F 2 "Pin_Headers:Pin_Header_Straight_1x05" H 5000 950 60  0001 C CNN
+F 3 "" H 5000 950 60  0000 C CNN
+	1    5000 950
+	0    -1   -1   0
+$EndComp
+Wire Wire Line
+	4800 1150 4800 1850
+Connection ~ 4800 1850
+Wire Wire Line
+	4900 1150 4900 1950
+Connection ~ 4900 1950
+Wire Wire Line
+	5000 1150 5000 1550
+Wire Wire Line
+	5000 1550 6900 1550
+Wire Wire Line
+	5100 1150 5100 1450
+Wire Wire Line
+	5100 1450 7000 1450
+Wire Wire Line
+	7000 1450 7000 1850
+Connection ~ 7000 1850
+Wire Wire Line
+	5200 1150 5200 1350
+Wire Wire Line
+	5200 1350 6700 1350
+Connection ~ 6700 1950
+Wire Wire Line
+	6900 1550 6900 2150
+Connection ~ 6900 2150
 $EndSCHEMATC

Commit message: Updated circuit diagram.
Parts:
- removed U3: TA48M033F, Transistors_TO-220:TO-220_Neutral123_Vertical, symbol LM7805CT
- added C3: 0.1u, Capacitors_ThroughHole:C_Disc_D3_P2.5, symbol C_Small
- added SP1: PiezoSpk, Connect:bornier2, symbol Crystal
- added U3: XC6202P332TB, Housings_TO-92:TO-92_Inline_Wide, symbol APE8865NL-33-HF-3
Connections:
- wire segments 57 -> 62
