File: KiCad/CarSpeedPulser.sch (KiCad schematic (older format))
At the start: 18 parts, among them P1 CONN_01X03, P2 CONN_01X05, Q1 2SK4017, SW1 RESET, SW2 UP, SW3 DOWN, U1 LPC810, U2 AE-AQM0802, U3 XC6202P332TB

Commit message: Removed pullup register. PULSE output is open drain.
Parts:
- removed R3: 10k, Resistors_ThroughHole:Resistor_Horizontal_RM10mm, symbol R
Connections:
- wire segments 62 -> 61
Changed lines of the file:
@@
 LIBS:contrib
 LIBS:valves
+LIBS:CarSpeedPulser-cache
 EELAYER 25 0
 EELAYER END
@@
 $EndComp
 $Comp
-L R R3
-U 1 1 554F2223
-P 3350 2800
-F 0 "R3" V 3430 2800 50  0000 C CNN
-F 1 "10k" V 3350 2800 50  0000 C CNN
-F 2 "Resistors_ThroughHole:Resistor_Horizontal_RM10mm" V 3280 2800 30  0001 C CNN
-F 3 "" H 3350 2800 30  0000 C CNN
-	1    3350 2800
-	1    0    0    -1
-$EndComp
-$Comp
 L R R2
 U 1 1 554F2D71
@@
 	2650 3450 3050 3450
 Wire Wire Line
-	3350 2950 3350 3250
-Wire Wire Line
-	3350 2650 3350 2500
+	3350 3200 3350 3250
 Wire Wire Line
 	3350 3900 3350 3650
@@
 Wire Wire Line
 	5100 3200 3350 3200
-Connection ~ 3350 3200
 Wire Wire Line
 	2950 2950 2950 1950
@@
 	8050 4200 8300 4200
 Connection ~ 8300 4200
-$Comp
-L +12V #PWR09
-U 1 1 554F1C57
-P 3350 2500
-F 0 "#PWR09" H 3350 2350 50  0001 C CNN
-F 1 "+12V" H 3350 2640 50  0000 C CNN
-F 2 "" H 3350 2500 60  0000 C CNN
-F 3 "" H 3350 2500 60  0000 C CNN
-	1    3350 2500
-	1    0    0    -1
-$EndComp
 Text Label 3500 3200 0    60   ~ 0
 PULSE
@@
 Connection ~ 4800 3300
 $Comp
-L +12V #PWR010
+L +12V #PWR09
 U 1 1 555EA485
 P 5100 2900
-F 0 "#PWR010" H 5100 2750 50  0001 C CNN
+F 0 "#PWR09" H 5100 2750 50  0001 C CNN
 F 1 "+12V" H 5100 3040 50  0000 C CNN
 F 2 "" H 5100 2900 60  0000 C CNN

Commit message: Replaced AE-AQM802 with AQM0802A-RN-GBW.
Parts:
- removed U2: AE-AQM0802, pulser:AE-AQM0802, symbol AE-AQM0802
- added C4, C5: 1u, Capacitors_ThroughHole:C_Disc_D3_P2.5, symbol C_Small
- added R4, R5: 10k, Resistors_ThroughHole:Resistor_Horizontal_RM10mm, symbol R
- added U2: AQM0802A-RN-GBW, pulser:AQM0802A-RN-GBW, symbol AQM0802A-RN-GBW
- SP1: footprint Connect:bornier2 -> Pin_Headers:Pin_Header_Straight_1x02
- renumbered R4 to R3
Connections:
- net labels added: SCL, SDA
- wire segments 61 -> 72
- no-connect marks 1 -> 0
Changed lines of the file:
@@
 EESchema Schematic File Version 2
 LIBS:LPC810
-LIBS:AE-AQM0802
+LIBS:AQM0802
 LIBS:power
 LIBS:device
@@
 L VDD #PWR04
 U 1 1 555A13C5
-P 7400 1550
-F 0 "#PWR04" H 7400 1400 50  0001 C CNN
-F 1 "VDD" H 7400 1700 50  0000 C CNN
-F 2 "" H 7400 1550 60  0000 C CNN
-F 3 "" H 7400 1550 60  0000 C CNN
-	1    7400 1550
+P 7900 900
+F 0 "#PWR04" H 7900 750 50  0001 C CNN
+F 1 "VDD" H 7900 1050 50  0000 C CNN
+F 2 "" H 7900 900 60  0000 C CNN
+F 3 "" H 7900 900 60  0000 C CNN
+	1    7900 900
 	1    0    0    -1
 $EndComp
@@
 $EndComp
 $Comp
-L AE-AQM0802 U2
-U 1 1 555A2C55
-P 8200 1850
-F 0 "U2" H 8200 1750 50  0000 C CNN
-F 1 "AE-AQM0802" H 8200 2200 50  0000 C CNN
-F 2 "pulser:AE-AQM0802" H 8200 1500 50  0001 C CNN
-F 3 "DOCUMENTATION" H 8200 1400 50  0001 C CNN
-	1    8200 1850
-	1    0    0    -1
-$EndComp
-NoConn ~ 7600 1750
-$Comp
 L PWR_FLAG #FLG06
 U 1 1 555A43B7
@@
 	1    0    0    -1
 $EndComp
-Connection ~ 8300 3850
-Wire Wire Line
-	8300 3750 8300 4300
-Wire Wire Line
-	8800 3850 8800 3700
-Wire Wire Line
-	7700 3850 8800 3850
-Wire Wire Line
-	7700 3700 7700 3850
-Connection ~ 8800 3400
-Wire Wire Line
-	8800 3250 8800 3500
-Wire Wire Line
-	8750 3400 8800 3400
-Connection ~ 7700 3400
-Wire Wire Line
-	7700 3400 7850 3400
-Wire Wire Line
-	7700 3150 7700 3500
-Wire Wire Line
-	2650 3450 3050 3450
-Wire Wire Line
-	3350 3200 3350 3250
-Wire Wire Line
-	3350 3900 3350 3650
-Wire Wire Line
-	2950 3250 2950 3500
-Wire Wire Line
-	2950 3800 2950 3900
-Wire Wire Line
-	4800 3900 2250 3900
-Connection ~ 3350 3900
-Connection ~ 2950 3450
-Wire Wire Line
-	4800 2200 4800 2150
-Wire Wire Line
-	4800 2150 5000 2150
-Wire Wire Line
-	4400 2200 4400 2050
-Wire Wire Line
-	4400 2050 5000 2050
-Wire Wire Line
-	4050 2200 4050 1850
-Wire Wire Line
-	4050 1850 5000 1850
-Wire Wire Line
-	5100 3200 3350 3200
-Wire Wire Line
-	2950 2950 2950 1950
-Wire Wire Line
-	2250 1950 5000 1950
-Wire Wire Line
-	4050 2800 4050 3000
-Wire Wire Line
-	4050 3000 4800 3000
-Wire Wire Line
-	4800 2800 4800 4050
-Wire Wire Line
-	4400 2800 4400 3000
-Connection ~ 4400 3000
-Connection ~ 4800 3000
-Wire Wire Line
-	6600 1950 6950 1950
-Wire Wire Line
-	6950 1350 6950 2650
-Wire Wire Line
-	7400 2050 7400 1550
-Wire Wire Line
-	6600 2050 7400 2050
-Wire Wire Line
-	6600 1850 7600 1850
-Wire Wire Line
-	7600 1650 7400 1650
-Connection ~ 7400 1650
-Wire Wire Line
-	6600 2150 7500 2150
-Wire Wire Line
-	7500 2150 7500 1950
-Wire Wire Line
-	7500 1950 7600 1950
-Wire Wire Line
-	7600 2050 7600 2250
-Wire Wire Line
-	7600 2250 6950 2250
-Wire Wire Line
-	7350 3200 7350 3250
-Wire Wire Line
-	7350 3250 7700 3250
-Connection ~ 7700 3250
-Connection ~ 4800 3900
-Connection ~ 6950 2250
 $Comp
 L LED D1
@@
 $EndComp
 $Comp
-L R R4
+L R R3
 U 1 1 555AA04E
 P 2250 2900
-F 0 "R4" V 2330 2900 50  0000 C CNN
+F 0 "R3" V 2330 2900 50  0000 C CNN
 F 1 "100" V 2250 2900 50  0000 C CNN
 F 2 "Resistors_ThroughHole:Resistor_Horizontal_RM10mm" V 2180 2900 30  0001 C CNN
@@
 	-1   0    0    1
 $EndComp
-Wire Wire Line
-	2250 2750 2250 1950
-Connection ~ 2950 1950
-Wire Wire Line
-	2250 3250 2250 3050
-Wire Wire Line
-	2250 3900 2250 3650
-Connection ~ 2950 3900
 $Comp
 L PWR_FLAG #FLG08
@@
 	1    0    0    -1
 $EndComp
-Wire Wire Line
-	8050 4200 8300 4200
-Connection ~ 8300 4200
 Text Label 3500 3200 0    60   ~ 0
 PULSE
@@
 	0    -1   -1   0
 $EndComp
-Wire Wire Line
-	4800 1150 4800 1850
-Connection ~ 4800 1850
-Wire Wire Line
-	4900 1150 4900 1950
-Connection ~ 4900 1950
-Wire Wire Line
-	5000 1150 5000 1550
-Wire Wire Line
-	5000 1550 7150 1550
-Wire Wire Line
-	5100 1150 5100 1450
-Wire Wire Line
-	5100 1450 7250 1450
-Wire Wire Line
-	7250 1450 7250 1850
-Connection ~ 7250 1850
-Wire Wire Line
-	5200 1150 5200 1350
-Wire Wire Line
-	5200 1350 6950 1350
-Connection ~ 6950 1950
-Wire Wire Line
-	7150 1550 7150 2150
-Connection ~ 7150 2150
 $Comp
 L Crystal SP1
@@
 F 0 "SP1" H 2650 3800 50  0000 C CNN
 F 1 "PiezoSpk" H 2650 3500 50  0000 C CNN
-F 2 "Connect:bornier2" H 2650 3650 60  0001 C CNN
+F 2 "Pin_Headers:Pin_Header_Straight_1x02" H 2650 3650 60  0001 C CNN
 F 3 "" H 2650 3650 60  0000 C CNN
 	1    2650 3650
 	0    1    1    0
 $EndComp
-Wire Wire Line
-	2650 3800 2650 3900
-Connection ~ 2650 3900
-Wire Wire Line
-	2650 3500 2650 3450
 $Comp
 L APE8865NL-33-HF-3 U3
@@
 	1    0    0    -1
 $EndComp
-Wire Wire Line
-	6700 2450 6700 2550
-Wire Wire Line
-	6700 2550 6950 2550
-Connection ~ 6950 2550
-Wire Wire Line
-	6700 2250 6700 2050
-Connection ~ 6700 2050
 $Comp
 L CONN_01X03 P1
@@
 	1    0    0    -1
 $EndComp
-Wire Wire Line
-	5100 3300 4800 3300
-Connection ~ 4800 3300
 $Comp
 L +12V #PWR09
@@
 	1    0    0    -1
 $EndComp
+$Comp
+L AQM0802A-RN-GBW U2
+U 1 1 563FF79A
+P 9250 1550
+F 0 "U2" H 9250 1000 50  0000 C CNN
+F 1 "AQM0802A-RN-GBW" H 9250 2200 50  0000 C CNN
+F 2 "pulser:AQM0802A-RN-GBW" H 9250 1000 50  0001 C CNN
+F 3 "DOCUMENTATION" H 9250 900 50  0001 C CNN
+	1    9250 1550
+	1    0    0    -1
+$EndComp
+Text Label 6550 1850 0    60   ~ 0
+SCL
+Text Label 6750 2150 0    60   ~ 0
+SDA
+$Comp
+L C_Small C5
+U 1 1 564021C2
+P 8400 1350
+F 0 "C5" H 8410 1420 50  0000 L CNN
+F 1 "1u" H 8410 1270 50  0000 L CNN
+F 2 "Capacitors_ThroughHole:C_Disc_D3_P2.5" H 8400 1350 60  0001 C CNN
+F 3 "" H 8400 1350 60  0000 C CNN
+	1    8400 1350
+	0    1    1    0
+$EndComp
+$Comp
+L C_Small C4
+U 1 1 5640246F
+P 8100 1250
+F 0 "C4" H 8110 1320 50  0000 L CNN
+F 1 "1u" H 8110 1170 50  0000 L CNN
+F 2 "Capacitors_ThroughHole:C_Disc_D3_P2.5" H 8100 1250 60  0001 C CNN
+F 3 "" H 8100 1250 60  0000 C CNN
+	1    8100 1250
+	0    1    1    0
+$EndComp
+Connection ~ 8300 3850
+Wire Wire Line
+	8300 3750 8300 4300
+Wire Wire Line
+	8800 3850 8800 3700
+Wire Wire Line
+	7700 3850 8800 3850
+Wire Wire Line
+	7700 3700 7700 3850
+Connection ~ 8800 3400
+Wire Wire Line
+	8800 3250 8800 3500
+Wire Wire Line
+	8750 3400 8800 3400
+Connection ~ 7700 3400
+Wire Wire Line
+	7700 3400 7850 3400
+Wire Wire Line
+	7700 3150 7700 3500
+Wire Wire Line
+	2650 3450 3050 3450
+Wire Wire Line
+	3350 3200 3350 3250
+Wire Wire Line
+	3350 3900 3350 3650
+Wire Wire Line
+	2950 3250 2950 3500
+Wire Wire Line
+	2950 3800 2950 3900
+Wire Wire Line
+	4800 3900 2250 3900
+Connection ~ 3350 3900
+Connection ~ 2950 3450
+Wire Wire Line
+	4800 2200 4800 2150
+Wire Wire Line
+	4800 2150 5000 2150
+Wire Wire Line
+	4400 2200 4400 2050
+Wire Wire Line
+	4400 2050 5000 2050
+Wire Wire Line
+	4050 2200 4050 1850
+Wire Wire Line
+	4050 1850 5000 1850
+Wire Wire Line
+	5100 3200 3350 3200
+Wire Wire Line
+	2950 2950 2950 1950
+Wire Wire Line
+	2250 1950 5000 1950
+Wire Wire Line
+	4050 2800 4050 3000
+Wire Wire Line
+	4050 3000 4800 3000
+Wire Wire Line
+	4800 2800 4800 4050
+Wire Wire Line
+	4400 2800 4400 3000
+Connection ~ 4400 3000
+Connection ~ 4800 3000
+Wire Wire Line
+	6950 1950 6600 1950
+Wire Wire Line
+	6950 1350 6950 2650
+Wire Wire Line
+	7900 2050 7900 900
+Wire Wire Line
+	6600 2050 7900 2050
+Wire Wire Line
+	6600 1850 8650 1850
+Wire Wire Line
+	7900 1550 8650 1550
+Wire Wire Line
+	6600 2150 8400 2150
+Wire Wire Line
+	7350 3200 7350 3250
+Wire Wire Line
+	7350 3250 7700 3250
+Connection ~ 7700 3250
+Connection ~ 4800 3900
+Wire Wire Line
+	2250 2750 2250 1950
+Connection ~ 2950 1950
+Wire Wire Line
+	2250 3250 2250 3050
+Wire Wire Line
+	2250 3900 2250 3650
+Connection ~ 2950 3900
+Wire Wire Line
+	8050 4200 8300 4200
+Connection ~ 8300 4200
+Wire Wire Line
+	4800 1150 4800 1850
+Connection ~ 4800 1850
+Wire Wire Line
+	4900 1150 4900 1950
+Connection ~ 4900 1950
+Wire Wire Line
+	5000 1150 5000 1550
+Wire Wire Line
+	5000 1550 7150 1550
+Wire Wire Line
+	5100 1150 5100 1450
+Wire Wire Line
+	5100 1450 6800 1450
+Wire Wire Line
+	6800 1450 6800 1850
+Connection ~ 6800 1850
+Wire Wire Line
+	5200 1150 5200 1350
+Wire Wire Line
+	5200 1350 6950 1350
+Connection ~ 6950 1950
+Wire Wire Line
+	7150 1550 7150 2150
+Connection ~ 7150 2150
+Wire Wire Line
+	2650 3800 2650 3900
+Connection ~ 2650 3900
+Wire Wire Line
+	2650 3500 2650 3450
+Wire Wire Line
+	6700 2450 6700 2550
+Wire Wire Line
+	6700 2550 6950 2550
+Connection ~ 6950 2550
+Wire Wire Line
+	6700 2250 6700 2050
+Connection ~ 6700 2050
+Wire Wire Line
+	5100 3300 4800 3300
+Connection ~ 4800 3300
 Wire Wire Line
 	5100 3100 5100 2900
+Wire Wire Line
+	6950 1650 8650 1650
+Wire Wire Line
+	8400 1750 8650 1750
+Wire Wire Line
+	8650 1250 8200 1250
+Wire Wire Line
+	7350 1250 8000 1250
+Wire Wire Line
+	8500 1350 8650 1350
+Wire Wire Line
+	8300 1350 8200 1350
+Wire Wire Line
+	8200 1350 8200 1450
+Wire Wire Line
+	8200 1450 8650 1450
+Wire Wire Line
+	8650 1950 8500 1950
+Wire Wire Line
+	8500 1950 8500 1550
+Connection ~ 8500 1550
+Wire Wire Line
+	8400 2150 8400 1750
+Connection ~ 7900 1550
+Connection ~ 6950 1650
+Connection ~ 7900 1250
+$Comp
+L R R4
+U 1 1 56404CAB
+P 7350 1450
+F 0 "R4" V 7430 1450 50  0000 C CNN
+F 1 "10k" V 7350 1450 50  0000 C CNN
+F 2 "Resistors_ThroughHole:Resistor_Horizontal_RM10mm" V 7280 1450 30  0001 C CNN
+F 3 "" H 7350 1450 30  0000 C CNN
+	1    7350 1450
+	-1   0    0    1
+$EndComp
+$Comp
+L R R5
+U 1 1 56404FAB
+P 7550 1450
+F 0 "R5" V 7630 1450 50  0000 C CNN
+F 1 "10k" V 7550 1450 50  0000 C CNN
+F 2 "Resistors_ThroughHole:Resistor_Horizontal_RM10mm" V 7480 1450 30  0001 C CNN
+F 3 "" H 7550 1450 30  0000 C CNN
+	1    7550 1450
+	-1   0    0    1
+$EndComp
+Wire Wire Line
+	7550 1600 7550 2050
+Connection ~ 7550 2050
+Wire Wire Line
+	7350 1600 7350 1850
+Connection ~ 7350 1850
+Wire Wire Line
+	7350 1300 7350 1250
+Wire Wire Line
+	7550 1300 7550 1250
+Connection ~ 7550 1250
 $EndSCHEMATC

Commit message: Changed footprint of a speaker.
Parts:
- SP1: footprint Pin_Headers:Pin_Header_Straight_1x02 -> Buzzers_Beepers:MagneticBuzzer_Kingstate_KCG0601
Changed lines of the file:
@@
 F 0 "SP1" H 2650 3800 50  0000 C CNN
 F 1 "PiezoSpk" H 2650 3500 50  0000 C CNN
-F 2 "Pin_Headers:Pin_Header_Straight_1x02" H 2650 3650 60  0001 C CNN
+F 2 "Buzzers_Beepers:MagneticBuzzer_Kingstate_KCG0601" H 2650 3650 60  0001 C CNN
 F 3 "" H 2650 3650 60  0000 C CNN
 	1    2650 3650

Commit message: Replaced voltage regulator to SMD type.
Parts:
- removed C2: 1u, Capacitors_ThroughHole:C_Disc_D3_P2.5, symbol CP_Small
- removed SP1: PiezoSpk, Buzzers_Beepers:MagneticBuzzer_Kingstate_KCG0601, symbol Crystal
- added C2: 1u, Capacitors_SMD:C_0805_HandSoldering, symbol C_Small
- C1, C4, C5: footprint Capacitors_ThroughHole:C_Disc_D3_P2.5 -> Capacitors_SMD:C_0805_HandSoldering
- C3: value 0.1u -> 1u; footprint Capacitors_ThroughHole:C_Disc_D3_P2.5 -> Capacitors_SMD:C_0805_HandSoldering
- D1: footprint LEDs:LED-3MM -> favorites:LED-1206
- Q1: value 2SK4017 -> RUE002N02; footprint Transistors_TO-220:TO-220_Neutral123_Vertical -> favorites:EMT3; symbol Q_NMOS_GDS -> Q_NMOS_SGD
- R1, R4, R5: footprint Resistors_ThroughHole:Resistor_Horizontal_RM10mm -> Resistors_SMD:R_0603_HandSoldering
- R2: value 100k -> 1M; footprint Resistors_ThroughHole:Resistor_Horizontal_RM10mm -> Resistors_SMD:R_0603_HandSoldering
- R3: value 100 -> 680; footprint Resistors_ThroughHole:Resistor_Horizontal_RM10mm -> Resistors_SMD:R_0603_HandSoldering
- U3: value XC6202P332TB -> NJU7223DL1-33; footprint Housings_TO-92:TO-92_Inline_Wide -> favorites:TO-252; symbol APE8865NL-33-HF-3 -> NJU7223DL1-33
Connections:
- net labels added: #RST, CAP1N, CAP1P, GATE, PIO0_2, PIO0_3, PIO0_4, VOUT, VSS
- wire segments 72 -> 70
Changed lines of the file:
@@
 EESchema Schematic File Version 2
 LIBS:LPC810
+LIBS:NJU7223DL1
 LIBS:AQM0802
 LIBS:power
@@
 LIBS:memory
 LIBS:xilinx
-LIBS:special
 LIBS:microcontrollers
 LIBS:dsp
@@
 $EndDescr
 $Comp
-L CP_Small C2
-U 1 1 554DA473
-P 8800 3600
-F 0 "C2" H 8810 3670 50  0000 L CNN
-F 1 "1u" H 8810 3520 50  0000 L CNN
-F 2 "Capacitors_ThroughHole:C_Disc_D3_P2.5" H 8800 3600 60  0001 C CNN
-F 3 "" H 8800 3600 60  0000 C CNN
-	1    8800 3600
-	1    0    0    -1
-$EndComp
-$Comp
 L C_Small C1
 U 1 1 554DA48F
@@
 F 0 "C1" H 7710 3670 50  0000 L CNN
 F 1 "1u" H 7710 3520 50  0000 L CNN
-F 2 "Capacitors_ThroughHole:C_Disc_D3_P2.5" H 7700 3600 60  0001 C CNN
+F 2 "Capacitors_SMD:C_0805_HandSoldering" H 7700 3600 60  0001 C CNN
 F 3 "" H 7700 3600 60  0000 C CNN
 	1    7700 3600
@@
 $EndComp
 $Comp
-L Q_NMOS_GDS Q1
+L Q_NMOS_SGD Q1
 U 1 1 554F19F4
 P 3250 3450
 F 0 "Q1" H 3550 3500 50  0000 R CNN
-F 1 "2SK4017" H 3750 3350 50  0000 R CNN
-F 2 "Transistors_TO-220:TO-220_Neutral123_Vertical" H 3450 3550 29  0001 C CNN
+F 1 "RUE002N02" H 3750 3350 50  0000 R CNN
+F 2 "favorites:EMT3" H 3450 3550 29  0001 C CNN
 F 3 "" H 3250 3450 60  0000 C CNN
 	1    3250 3450
@@
 F 0 "R1" V 3030 3100 50  0000 C CNN
 F 1 "1k" V 2950 3100 50  0000 C CNN
-F 2 "Resistors_ThroughHole:Resistor_Horizontal_RM10mm" V 2880 3100 30  0001 C CNN
+F 2 "Resistors_SMD:R_0603_HandSoldering" V 2880 3100 30  0001 C CNN
 F 3 "" H 2950 3100 30  0000 C CNN
 	1    2950 3100
@@
 P 2950 3650
 F 0 "R2" V 3030 3650 50  0000 C CNN
-F 1 "100k" V 2950 3650 50  0000 C CNN
-F 2 "Resistors_ThroughHole:Resistor_Horizontal_RM10mm" V 2880 3650 30  0001 C CNN
+F 1 "1M" V 2950 3650 50  0000 C CNN
+F 2 "Resistors_SMD:R_0603_HandSoldering" V 2880 3650 30  0001 C CNN
 F 3 "" H 2950 3650 30  0000 C CNN
 	1    2950 3650
@@
 F 0 "D1" H 2250 3550 50  0000 C CNN
 F 1 "LED" H 2250 3350 50  0000 C CNN
-F 2 "LEDs:LED-3MM" H 2250 3450 60  0001 C CNN
+F 2 "favorites:LED-1206" H 2250 3450 60  0001 C CNN
 F 3 "" H 2250 3450 60  0000 C CNN
 	1    2250 3450
@@
 P 2250 2900
 F 0 "R3" V 2330 2900 50  0000 C CNN
-F 1 "100" V 2250 2900 50  0000 C CNN
-F 2 "Resistors_ThroughHole:Resistor_Horizontal_RM10mm" V 2180 2900 30  0001 C CNN
+F 1 "680" V 2250 2900 50  0000 C CNN
+F 2 "Resistors_SMD:R_0603_HandSoldering" V 2180 2900 30  0001 C CNN
 F 3 "" H 2250 2900 30  0000 C CNN
 	1    2250 2900
@@
 $EndComp
 $Comp
-L Crystal SP1
-U 1 1 555B3095
-P 2650 3650
-F 0 "SP1" H 2650 3800 50  0000 C CNN
-F 1 "PiezoSpk" H 2650 3500 50  0000 C CNN
-F 2 "Buzzers_Beepers:MagneticBuzzer_Kingstate_KCG0601" H 2650 3650 60  0001 C CNN
-F 3 "" H 2650 3650 60  0000 C CNN
-	1    2650 3650
-	0    1    1    0
-$EndComp
-$Comp
-L APE8865NL-33-HF-3 U3
+L NJU7223DL1-33 U3
 U 1 1 555B31B5
 P 8300 3450
 F 0 "U3" H 8000 3700 40  0000 C CNN
-F 1 "XC6202P332TB" H 8300 3650 40  0000 C CNN
-F 2 "Housings_TO-92:TO-92_Inline_Wide" H 8300 3550 35  0000 C CIN
+F 1 "NJU7223DL1-33" H 8300 3650 40  0000 C CNN
+F 2 "favorites:TO-252" H 8300 3550 35  0000 C CIN
 F 3 "" H 8300 3450 60  0000 C CNN
 	1    8300 3450
@@
 P 6700 2350
 F 0 "C3" H 6710 2420 50  0000 L CNN
-F 1 "0.1u" H 6710 2270 50  0000 L CNN
-F 2 "Capacitors_ThroughHole:C_Disc_D3_P2.5" H 6700 2350 60  0001 C CNN
+F 1 "1u" H 6710 2270 50  0000 L CNN
+F 2 "Capacitors_SMD:C_0805_HandSoldering" H 6700 2350 60  0001 C CNN
 F 3 "" H 6700 2350 60  0000 C CNN
 	1    6700 2350
@@
 	1    0    0    -1
 $EndComp
-Text Label 6550 1850 0    60   ~ 0
+Text Label 7050 1850 0    60   ~ 0
 SCL
 Text Label 6750 2150 0    60   ~ 0
@@
 L C_Small C5
 U 1 1 564021C2
-P 8400 1350
-F 0 "C5" H 8410 1420 50  0000 L CNN
-F 1 "1u" H 8410 1270 50  0000 L CNN
-F 2 "Capacitors_ThroughHole:C_Disc_D3_P2.5" H 8400 1350 60  0001 C CNN
-F 3 "" H 8400 1350 60  0000 C CNN
-	1    8400 1350
+P 8300 1350
+F 0 "C5" H 8310 1420 50  0000 L CNN
+F 1 "1u" H 8310 1270 50  0000 L CNN
+F 2 "Capacitors_SMD:C_0805_HandSoldering" H 8300 1350 60  0001 C CNN
+F 3 "" H 8300 1350 60  0000 C CNN
+	1    8300 1350
 	0    1    1    0
 $EndComp
@@
 F 0 "C4" H 8110 1320 50  0000 L CNN
 F 1 "1u" H 8110 1170 50  0000 L CNN
-F 2 "Capacitors_ThroughHole:C_Disc_D3_P2.5" H 8100 1250 60  0001 C CNN
+F 2 "Capacitors_SMD:C_0805_HandSoldering" H 8100 1250 60  0001 C CNN
 F 3 "" H 8100 1250 60  0000 C CNN
 	1    8100 1250
@@
 	7700 3150 7700 3500
 Wire Wire Line
-	2650 3450 3050 3450
+	2950 3450 3050 3450
 Wire Wire Line
 	3350 3200 3350 3250
@@
 Connection ~ 7150 2150
 Wire Wire Line
-	2650 3800 2650 3900
-Connection ~ 2650 3900
-Wire Wire Line
-	2650 3500 2650 3450
-Wire Wire Line
 	6700 2450 6700 2550
 Wire Wire Line
@@
 	7350 1250 8000 1250
 Wire Wire Line
-	8500 1350 8650 1350
-Wire Wire Line
-	8300 1350 8200 1350
+	8400 1350 8650 1350
+Wire Wire Line
+	8200 1350 8200 1350
 Wire Wire Line
 	8200 1350 8200 1450
@@
 F 0 "R4" V 7430 1450 50  0000 C CNN
 F 1 "10k" V 7350 1450 50  0000 C CNN
-F 2 "Resistors_ThroughHole:Resistor_Horizontal_RM10mm" V 7280 1450 30  0001 C CNN
+F 2 "Resistors_SMD:R_0603_HandSoldering" V 7280 1450 30  0001 C CNN
 F 3 "" H 7350 1450 30  0000 C CNN
 	1    7350 1450
@@
 F 0 "R5" V 7630 1450 50  0000 C CNN
 F 1 "10k" V 7550 1450 50  0000 C CNN
-F 2 "Resistors_ThroughHole:Resistor_Horizontal_RM10mm" V 7480 1450 30  0001 C CNN
+F 2 "Resistors_SMD:R_0603_HandSoldering" V 7480 1450 30  0001 C CNN
 F 3 "" H 7550 1450 30  0000 C CNN
 	1    7550 1450
@@
 $EndComp
 Wire Wire Line
-	7550 1600 7550 2050
-Connection ~ 7550 2050
-Wire Wire Line
 	7350 1600 7350 1850
 Connection ~ 7350 1850
@@
 	7550 1300 7550 1250
 Connection ~ 7550 1250
+$Comp
+L C_Small C2
+U 1 1 56481F6D
+P 8800 3600
+F 0 "C2" H 8810 3670 50  0000 L CNN
+F 1 "1u" H 8810 3520 50  0000 L CNN
+F 2 "Capacitors_SMD:C_0805_HandSoldering" H 8800 3600 60  0001 C CNN
+F 3 "" H 8800 3600 60  0000 C CNN
+	1    8800 3600
+	1    0    0    -1
+$EndComp
+Text Label 4150 1850 0    60   ~ 0
+#RST
+Text Label 4200 1950 0    60   ~ 0
+PIO0_4
+Text Label 4500 2050 0    60   ~ 0
+PIO0_3
+Text Label 4850 2150 0    60   ~ 0
+PIO0_2
+Text Label 6750 2050 0    60   ~ 0
+VDD
+Text Label 6700 1950 0    60   ~ 0
+VSS
+Text Label 4300 3900 0    60   ~ 0
+GND
+Text Label 2950 3400 0    60   ~ 0
+GATE
+Text Label 8250 1250 0    60   ~ 0
+VOUT
+Text Label 8450 1350 0    60   ~ 0
+CAP1N
+Text Label 8500 1450 0    60   ~ 0
+CAP1P
+Wire Wire Line
+	7550 1600 7550 2150
+Connection ~ 7550 2150
 $EndSCHEMATC

Commit message: Added diodes, registers and a voltage detector.
Parts:
- added D2, D3: 1N4148W, Diodes_SMD:SOD-123, symbol D
- added R6: 1M, Resistors_SMD:R_0603_HandSoldering, symbol R
- added U4: BD45231G, favorites:SSOP5_Handsoldering, symbol BD45231G
Connections:
- net labels added: D, Vin
- net labels removed: GND
- wire segments 70 -> 85

Commit message: Updated KiCad parts library
Parts:
- D1: footprint favorites:LED-1206 -> LEDs:LED_1206_HandSoldering
- P1: symbol CONN_01X03 -> Conn_01x03
- P2: symbol CONN_01X05 -> Conn_01x05
- SW1, SW2, SW3: symbol SW_PUSH -> SW_Push
Changed lines of the file:
@@
 EESchema Schematic File Version 2
+LIBS:CarSpeedPulser-rescue
 LIBS:LPC810
 LIBS:NJU7223DL1
@@
 LIBS:valves
 LIBS:favorites
+LIBS:switches
 LIBS:CarSpeedPulser-cache
 EELAYER 25 0
@@
 $EndComp
 $Comp
-L SW_PUSH SW3
+L SW_Push SW3
 U 1 1 554F7940
 P 5900 2550
@@
 $EndComp
 $Comp
-L SW_PUSH SW2
+L SW_Push SW2
 U 1 1 554F79EC
 P 5500 2550
@@
 $EndComp
 $Comp
-L SW_PUSH SW1
+L SW_Push SW1
 U 1 1 5559FDDD
 P 5150 2550
@@
 F 0 "D1" H 3650 3600 50  0000 C CNN
 F 1 "LED" H 3650 3400 50  0000 C CNN
-F 2 "favorites:LED-1206" H 3650 3500 60  0001 C CNN
+F 2 "LEDs:LED_1206_HandSoldering" H 3650 3500 60  0001 C CNN
 F 3 "" H 3650 3500 60  0000 C CNN
 	1    3650 3500
@@
 PULSE
 $Comp
-L CONN_01X05 P2
+L Conn_01x05 P2
 U 1 1 5559F1FE
 P 6100 1000
@@
 $EndComp
 $Comp
-L CONN_01X03 P1
+L Conn_01x03 P1
 U 1 1 555E9DB4
 P 6400 3250
@@
 Connection ~ 4050 3500
 Wire Wire Line
-	5900 2250 5900 2200
+	5900 2350 5900 2200
 Wire Wire Line
 	5900 2200 6100 2200
 Wire Wire Line
-	5500 2250 5500 2100
+	5500 2350 5500 2100
 Wire Wire Line
 	5500 2100 6100 2100
 Wire Wire Line
-	5150 1600 5150 2250
+	5150 1600 5150 2350
 Wire Wire Line
 	5150 1900 6100 1900
@@
 	3650 2000 6100 2000
 Wire Wire Line
-	5150 2850 5150 3050
+	5150 2750 5150 3050
 Wire Wire Line
 	5150 3050 5900 3050
 Wire Wire Line
-	5900 2850 5900 3950
-Wire Wire Line
-	5500 2850 5500 3050
+	5900 2750 5900 3950
+Wire Wire Line
+	5500 2750 5500 3050
 Connection ~ 5500 3050
 Connection ~ 5900 3050
@@
 Connection ~ 4050 2000
 Wire Wire Line
-	3650 3300 3650 3100
-Wire Wire Line
-	3650 3950 3650 3700
+	3650 3350 3650 3100
+Wire Wire Line
+	3650 3950 3650 3650
 Connection ~ 4050 3950
 Connection ~ 2600 3100
@@
 Connection ~ 5600 1900
 $Comp
-L VDD #PWR?
+L VDD #PWR08
 U 1 1 56A733F9
 P 4700 1200
-F 0 "#PWR?" H 4700 1050 50  0001 C CNN
+F 0 "#PWR08" H 4700 1050 50  0001 C CNN
 F 1 "VDD" H 4700 1350 50  0000 C CNN
 F 2 "" H 4700 1200 60  0000 C CNN

Commit message: Replaced 3.3V regulator
Parts:
- D2: symbol D -> 1N4148
- U3: value NJU7223DL1-33 -> NJM78L33SU3; footprint favorites:TO-252 -> TO_SOT_Packages_SMD:SOT-89-3_Handsoldering; symbol NJU7223DL1-33 -> AP2204RB-3.3
Connections:
- wire segments 85 -> 86
