File: KiCad/CarSpeedPulser.sch (KiCad schematic (older format))
At the start: 24 parts, among them P1 CONN_01X03, P2 CONN_01X05, Q1 RUE002N02, SW1 RESET, SW2 UP, SW3 DOWN, U1 LPC810, U2 AQM0802A-RN-GBW, U3 NJM78L33SU3, U4 BD45231G

Commit message: Replaced voltage detector
Parts:
- U4: value BD45231G -> R3111N211A; footprint favorites:SSOP5_Handsoldering -> TO_SOT_Packages_SMD:SOT-23-5_HandSoldering; symbol BD45231G -> R3111xxxx
Connections:
- wire segments 86 -> 85
Changed lines of the file:
@@
 LIBS:contrib
 LIBS:valves
-LIBS:favorites
 LIBS:switches
 LIBS:diode
+LIBS:R3111xxxx
 LIBS:CarSpeedPulser-cache
 EELAYER 25 0
@@
 L VDD #PWR03
 U 1 1 555A148D
-P 3100 2150
-F 0 "#PWR03" H 3100 2000 50  0001 C CNN
-F 1 "VDD" H 3100 2300 50  0000 C CNN
-F 2 "" H 3100 2150 60  0000 C CNN
-F 3 "" H 3100 2150 60  0000 C CNN
-	1    3100 2150
+P 3100 1150
+F 0 "#PWR03" H 3100 1000 50  0001 C CNN
+F 1 "VDD" H 3100 1300 50  0000 C CNN
+F 2 "" H 3100 1150 60  0000 C CNN
+F 3 "" H 3100 1150 60  0000 C CNN
+	1    3100 1150
 	1    0    0    -1
 $EndComp
@@
 $EndComp
 $Comp
-L BD45231G U4
+L R3111xxxx U4
 U 1 1 56A7058F
 P 4200 1500
-F 0 "U4" H 4200 1750 60  0000 C CNN
-F 1 "BD45231G" H 4200 1250 60  0000 C CNN
-F 2 "favorites:SSOP5_Handsoldering" H 4200 1500 60  0001 C CNN
-F 3 "" H 4200 1500 60  0000 C CNN
+F 0 "U4" H 4200 1800 60  0000 C CNN
+F 1 "R3111N211A" H 4200 1200 60  0000 C CNN
+F 2 "TO_SOT_Packages_SMD:SOT-23-5_HandSoldering" H 4200 1500 60  0001 C CNN
+F 3 "http://akizukidenshi.com/download/ds/ricoh/r3111x-j.pdf" H 4200 1500 60  0001 C CNN
 	1    4200 1500
 	1    0    0    -1
@@
 $EndComp
 $Comp
-L VDD #PWR07
-U 1 1 56A733F9
-P 4700 1200
-F 0 "#PWR07" H 4700 1050 50  0001 C CNN
-F 1 "VDD" H 4700 1350 50  0000 C CNN
-F 2 "" H 4700 1200 60  0000 C CNN
-F 3 "" H 4700 1200 60  0000 C CNN
-	1    4700 1200
-	1    0    0    -1
-$EndComp
-$Comp
-L PWR_FLAG #FLG08
+L PWR_FLAG #FLG07
 U 1 1 59C9EC89
 P 2200 2150
-F 0 "#FLG08" H 2200 2245 50  0001 C CNN
+F 0 "#FLG07" H 2200 2245 50  0001 C CNN
 F 1 "PWR_FLAG" H 2200 2330 50  0000 C CNN
 F 2 "" H 2200 2150 60  0000 C CNN
@@
 Connection ~ 3100 2300
 Wire Wire Line
-	3100 2150 3100 2400
+	3100 1150 3100 2400
 Wire Wire Line
 	2900 2300 3100 2300
@@
 	5500 2100 6100 2100
 Wire Wire Line
-	5150 1600 5150 2350
+	5150 1050 5150 2350
 Wire Wire Line
 	5150 1900 6100 1900
@@
 Wire Wire Line
 	6300 1200 6300 1400
-Wire Wire Line
-	4550 1400 5600 1400
 Wire Wire Line
 	6300 1400 8050 1400
@@
 	6100 3350 6200 3350
 Wire Wire Line
-	3300 1600 3850 1600
-Wire Wire Line
-	3300 1400 3300 3950
+	3300 1600 3600 1600
 Connection ~ 3300 3950
-Wire Wire Line
-	4550 1600 5150 1600
 Connection ~ 5150 1900
-Wire Wire Line
-	3850 1400 3300 1400
-Connection ~ 3300 1600
-Wire Wire Line
-	3850 1500 3300 1500
-Connection ~ 3300 1500
-Wire Wire Line
-	5600 1400 5600 1500
 Wire Wire Line
 	5600 1800 5600 1900
 Connection ~ 5600 1900
-Wire Wire Line
-	4700 1200 4700 1400
-Connection ~ 4700 1400
 Wire Wire Line
 	2200 2150 2200 2300
@@
 	1150 2050 1150 2300
 $Comp
-L PWR_FLAG #FLG09
+L PWR_FLAG #FLG08
 U 1 1 555A43B7
 P 1150 2050
-F 0 "#FLG09" H 1150 2145 50  0001 C CNN
+F 0 "#FLG08" H 1150 2145 50  0001 C CNN
 F 1 "PWR_FLAG" H 1150 2230 50  0000 C CNN
 F 2 "" H 1150 2050 60  0000 C CNN
@@
 	1    0    0    -1
 $EndComp
+Wire Wire Line
+	3300 1600 3300 3950
+$Comp
+L VDD #PWR09
+U 1 1 56A733F9
+P 5600 1100
+F 0 "#PWR09" H 5600 950 50  0001 C CNN
+F 1 "VDD" H 5600 1250 50  0000 C CNN
+F 2 "" H 5600 1100 60  0000 C CNN
+F 3 "" H 5600 1100 60  0000 C CNN
+	1    5600 1100
+	1    0    0    -1
+$EndComp
+Wire Wire Line
+	3600 1400 3550 1400
+Wire Wire Line
+	3550 1400 3550 1050
+Wire Wire Line
+	3550 1050 5150 1050
+Wire Wire Line
+	5600 1100 5600 1500
+Wire Wire Line
+	3600 1500 3100 1500
+Connection ~ 3100 1500
 $EndSCHEMATC
