File: KiCad/CarSpeedPulser.sch (KiCad schematic (older format))
At the start: 24 parts, among them P1 CONN_01X03, P2 CONN_01X05, Q1 RUE002N02, SW1 RESET, SW2 UP, SW3 DOWN, U1 LPC810, U2 AQM0802A-RN-GBW, U3 NJM78L33SU3, U4 R3111N211A

Commit message: Migrated to KiCad 5.0
Parts:
- C1, C2, C3, C4, C5: symbol C_Small -> device:C_Small
- D1: footprint LEDs:LED_1206_HandSoldering -> LED_SMD:LED_1206_3216Metric_Pad1.07x1.80mm_HandSolder; symbol LED -> device:LED
- D2: symbol 1N4148 -> diode:1N4148
- D3: symbol D -> device:D
- P1: symbol Conn_01x03 -> CarSpeedPulser-rescue:Conn_01x03
- P2: symbol Conn_01x05 -> CarSpeedPulser-rescue:Conn_01x05
- Q1: symbol Q_NMOS_SGD -> device:Q_NMOS_SGD
- R1, R2, R3, R4, R5: footprint Resistors_SMD:R_0603_HandSoldering -> Resistor_SMD:R_0603_1608Metric_Pad0.84x1.00mm_HandSolder; symbol R -> device:R
- R6: symbol R -> device:R
- SW1, SW2, SW3: symbol SW_Push -> CarSpeedPulser-rescue:SW_Push
- U1: footprint Sockets_DIP:DIP-8__300 -> Package_DIP:DIP-8_W7.62mm; symbol LPC810 -> LPC810:LPC810
- U2: symbol AQM0802A-RN-GBW -> AQM0802:AQM0802A-RN-GBW
- U3: footprint TO_SOT_Packages_SMD:SOT-89-3_Handsoldering -> Package_TO_SOT_SMD:SOT-89-3_Handsoldering; symbol AP2204RB-3.3 -> regul:AP2204RB-3.3
- U4: footprint TO_SOT_Packages_SMD:SOT-23-5_HandSoldering -> Package_TO_SOT_SMD:SOT-23-5_HandSoldering; symbol R3111xxxx -> R3111xxxx:R3111xxxx
Connections:
- wire segments 85 -> 120
